File: busboard_20cm/busboard_20cm.kicad_pcb (KiCad board)
At the start: 2 copper layers, 200 x 30 mm, 20 parts, among them J101 Conn_02x03_Odd_Even, J102 Conn_02x03_Odd_Even, J103 Conn_02x08_Odd_Even, J104 Conn_02x08_Odd_Even, J105 Conn_02x08_Odd_Even, J106 Conn_02x08_Odd_Even, J107 Conn_02x08_Odd_Even, J108 Conn_02x08_Odd_Even, J109 Conn_02x08_Odd_Even, J110 Conn_02x08_Odd_Even, J111 Conn_02x08_Odd_Even, J112 Conn_02x08_Odd_Even

Commit message: other connectors
Parts:
- J101, J102: footprint Connector_Molex:Molex_Mega-Fit_76825-0006_2x03_P5.70mm_Horizontal -> Connector_Molex:Molex_Mini-Fit_Jr_5569-06A2_2x03_P4.20mm_Horizontal
- moved J102 161.6 mm to (235.7, 60.8), turned to -90 degrees
- moved J110 156.0 mm to (78.2, 56.1)
- moved J101 14.2 mm to (64.3, 69.2), turned to 90 degrees

Commit message: 20cm busboard PCB
Parts:
- added C101: 100uF/25V, Capacitor_SMD:CP_Elec_6.3x7.7, F.Cu at (63.0, 54.0)
- added C102: 100uF/25V, Capacitor_SMD:CP_Elec_6.3x7.7, F.Cu at (63.0, 76.0)
- added C103: 100uF/25V, Capacitor_SMD:CP_Elec_6.3x7.7, F.Cu at (118.5, 63.7)
- added D101: RED, LED_SMD:LED_0603_1608Metric, F.Cu at (71.0, 59.0)
- added D102: RED, LED_SMD:LED_0603_1608Metric, F.Cu at (71.0, 69.0)
- added D103: RED, LED_SMD:LED_0603_1608Metric, F.Cu at (71.0, 64.0)
- added R101: 1k, Resistor_SMD:R_0603_1608Metric, F.Cu at (71.0, 61.0)
- added R102: 1k, Resistor_SMD:R_0603_1608Metric, F.Cu at (71.0, 71.0)
- added R103: 1k, Resistor_SMD:R_0603_1608Metric, F.Cu at (71.0, 66.0)
- J101, J102: value Conn_02x03_Odd_Even -> Conn_02x03_Top_Bottom
- moved J102 5.01 mm to (240.7, 60.5)
- moved J101 4.28 mm to (60.0, 69.2)
Connections:
- J101 pad 1: unconnected-(J101-Pad1) -> GND
- J101 pad 2: unconnected-(J101-Pad2) -> GND
- J101 pad 3: unconnected-(J101-Pad3) -> GND
- J101 pad 4: unconnected-(J101-Pad4) -> -12V
- J101 pad 5: unconnected-(J101-Pad5) -> +12V
- J101 pad 6: unconnected-(J101-Pad6) -> +5V
- J102 pad 1: unconnected-(J102-Pad1) -> GND
- J102 pad 2: unconnected-(J102-Pad2) -> GND
- J102 pad 3: unconnected-(J102-Pad3) -> GND
- J102 pad 4: unconnected-(J102-Pad4) -> +5V
- J102 pad 5: unconnected-(J102-Pad5) -> +12V
- J102 pad 6: unconnected-(J102-Pad6) -> -12V
- J103 pad 10: unconnected-(J103-Pad10) -> GND
- J103 pad 11: unconnected-(J103-Pad11) -> GND
- J103 pad 12: unconnected-(J103-Pad12) -> GND
- J103 pad 13: unconnected-(J103-Pad13) -> GND
- J103 pad 14: unconnected-(J103-Pad14) -> GND
- J103 pad 15: unconnected-(J103-Pad15) -> -12V
- J103 pad 16: unconnected-(J103-Pad16) -> -12V
- J103 pad 5: unconnected-(J103-Pad5) -> +5V
- J103 pad 6: unconnected-(J103-Pad6) -> +5V
- J103 pad 7: unconnected-(J103-Pad7) -> +12V
- J103 pad 8: unconnected-(J103-Pad8) -> +12V
- J103 pad 9: unconnected-(J103-Pad9) -> GND
- J104 pad 10: unconnected-(J104-Pad10) -> GND
- J104 pad 11: unconnected-(J104-Pad11) -> GND
- J104 pad 12: unconnected-(J104-Pad12) -> GND
- J104 pad 13: unconnected-(J104-Pad13) -> GND
- J104 pad 14: unconnected-(J104-Pad14) -> GND
- J104 pad 15: unconnected-(J104-Pad15) -> -12V
- J104 pad 16: unconnected-(J104-Pad16) -> -12V
- J104 pad 5: unconnected-(J104-Pad5) -> +5V
- J104 pad 6: unconnected-(J104-Pad6) -> +5V
- J104 pad 7: unconnected-(J104-Pad7) -> +12V
- J104 pad 8: unconnected-(J104-Pad8) -> +12V
- J104 pad 9: unconnected-(J104-Pad9) -> GND
- J105 pad 10: unconnected-(J105-Pad10) -> GND
- J105 pad 11: unconnected-(J105-Pad11) -> GND
- J105 pad 12: unconnected-(J105-Pad12) -> GND
- J105 pad 13: unconnected-(J105-Pad13) -> GND
- J105 pad 14: unconnected-(J105-Pad14) -> GND
- J105 pad 15: unconnected-(J105-Pad15) -> -12V
- J105 pad 16: unconnected-(J105-Pad16) -> -12V
- J105 pad 5: unconnected-(J105-Pad5) -> +5V
- J105 pad 6: unconnected-(J105-Pad6) -> +5V
- J105 pad 7: unconnected-(J105-Pad7) -> +12V
- J105 pad 8: unconnected-(J105-Pad8) -> +12V
- J105 pad 9: unconnected-(J105-Pad9) -> GND
- J106 pad 10: unconnected-(J106-Pad10) -> GND
- J106 pad 11: unconnected-(J106-Pad11) -> GND
- J106 pad 12: unconnected-(J106-Pad12) -> GND
- J106 pad 13: unconnected-(J106-Pad13) -> GND
- J106 pad 14: unconnected-(J106-Pad14) -> GND
- J106 pad 15: unconnected-(J106-Pad15) -> -12V
- J106 pad 16: unconnected-(J106-Pad16) -> -12V
- J106 pad 5: unconnected-(J106-Pad5) -> +5V
- J106 pad 6: unconnected-(J106-Pad6) -> +5V
- J106 pad 7: unconnected-(J106-Pad7) -> +12V
- J106 pad 8: unconnected-(J106-Pad8) -> +12V
- J106 pad 9: unconnected-(J106-Pad9) -> GND
- J107 pad 10: unconnected-(J107-Pad10) -> GND
- J107 pad 11: unconnected-(J107-Pad11) -> GND
- J107 pad 12: unconnected-(J107-Pad12) -> GND
- J107 pad 13: unconnected-(J107-Pad13) -> GND
- J107 pad 14: unconnected-(J107-Pad14) -> GND
- J107 pad 15: unconnected-(J107-Pad15) -> -12V
- J107 pad 16: unconnected-(J107-Pad16) -> -12V
- J107 pad 5: unconnected-(J107-Pad5) -> +5V
- J107 pad 6: unconnected-(J107-Pad6) -> +5V
- J107 pad 7: unconnected-(J107-Pad7) -> +12V
- J107 pad 8: unconnected-(J107-Pad8) -> +12V
- J107 pad 9: unconnected-(J107-Pad9) -> GND
- J108 pad 10: unconnected-(J108-Pad10) -> GND
- J108 pad 11: unconnected-(J108-Pad11) -> GND
- J108 pad 12: unconnected-(J108-Pad12) -> GND
- J108 pad 13: unconnected-(J108-Pad13) -> GND
- J108 pad 14: unconnected-(J108-Pad14) -> GND
- J108 pad 15: unconnected-(J108-Pad15) -> -12V
- J108 pad 16: unconnected-(J108-Pad16) -> -12V
- J108 pad 5: unconnected-(J108-Pad5) -> +5V
- J108 pad 6: unconnected-(J108-Pad6) -> +5V
- J108 pad 7: unconnected-(J108-Pad7) -> +12V
- J108 pad 8: unconnected-(J108-Pad8) -> +12V
- J108 pad 9: unconnected-(J108-Pad9) -> GND
- J109 pad 10: unconnected-(J109-Pad10) -> GND
- J109 pad 11: unconnected-(J109-Pad11) -> GND
- J109 pad 12: unconnected-(J109-Pad12) -> GND
- J109 pad 13: unconnected-(J109-Pad13) -> GND
- J109 pad 14: unconnected-(J109-Pad14) -> GND
- J109 pad 15: unconnected-(J109-Pad15) -> -12V
- J109 pad 16: unconnected-(J109-Pad16) -> -12V
- J109 pad 5: unconnected-(J109-Pad5) -> +5V
- J109 pad 6: unconnected-(J109-Pad6) -> +5V
- J109 pad 7: unconnected-(J109-Pad7) -> +12V
- J109 pad 8: unconnected-(J109-Pad8) -> +12V
- J109 pad 9: unconnected-(J109-Pad9) -> GND
- J110 pad 10: unconnected-(J110-Pad10) -> GND
- J110 pad 11: unconnected-(J110-Pad11) -> GND
- J110 pad 12: unconnected-(J110-Pad12) -> GND
- J110 pad 13: unconnected-(J110-Pad13) -> GND
- J110 pad 14: unconnected-(J110-Pad14) -> GND
- J110 pad 15: unconnected-(J110-Pad15) -> -12V
- J110 pad 16: unconnected-(J110-Pad16) -> -12V
- J110 pad 5: unconnected-(J110-Pad5) -> +5V
- J110 pad 6: unconnected-(J110-Pad6) -> +5V
- J110 pad 7: unconnected-(J110-Pad7) -> +12V
- J110 pad 8: unconnected-(J110-Pad8) -> +12V
- J110 pad 9: unconnected-(J110-Pad9) -> GND
- J111 pad 10: unconnected-(J111-Pad10) -> GND
- J111 pad 11: unconnected-(J111-Pad11) -> GND
- J111 pad 12: unconnected-(J111-Pad12) -> GND
- J111 pad 13: unconnected-(J111-Pad13) -> GND
- J111 pad 14: unconnected-(J111-Pad14) -> GND
- J111 pad 15: unconnected-(J111-Pad15) -> -12V
- J111 pad 16: unconnected-(J111-Pad16) -> -12V
- J111 pad 5: unconnected-(J111-Pad5) -> +5V
- J111 pad 6: unconnected-(J111-Pad6) -> +5V
- J111 pad 7: unconnected-(J111-Pad7) -> +12V
- J111 pad 8: unconnected-(J111-Pad8) -> +12V
- J111 pad 9: unconnected-(J111-Pad9) -> GND
- J112 pad 10: unconnected-(J112-Pad10) -> GND
- J112 pad 11: unconnected-(J112-Pad11) -> GND
- J112 pad 12: unconnected-(J112-Pad12) -> GND
- J112 pad 13: unconnected-(J112-Pad13) -> GND
- J112 pad 14: unconnected-(J112-Pad14) -> GND
- J112 pad 15: unconnected-(J112-Pad15) -> -12V
- J112 pad 16: unconnected-(J112-Pad16) -> -12V
- J112 pad 5: unconnected-(J112-Pad5) -> +5V
- J112 pad 6: unconnected-(J112-Pad6) -> +5V
- J112 pad 7: unconnected-(J112-Pad7) -> +12V
- J112 pad 8: unconnected-(J112-Pad8) -> +12V
- J112 pad 9: unconnected-(J112-Pad9) -> GND
Routing:
- net -12V: track 0.00 -> 195.8 mm
- net +12V: track 0.00 -> 182.8 mm
- net +5V: track 0.00 -> 182.5 mm
- net Net-(D103-Pad1): track 0.00 -> 2.02 mm
- net Net-(D102-Pad1): track 0.00 -> 2.02 mm
- net Net-(D101-Pad1): track 0.00 -> 2.02 mm
- net GND: vias 0 -> 68
- added copper zone on B.Cu, net GND
- added copper zone on F.Cu, net GND
